File: bodenfeuchte.sch (EAGLE design)
At the start: 16 parts, among them IC1 74HC14D, IC2 HT7333

Commit message: - new version of board - added trim resistor (500KΩ) to adjust cap. frequency (works like a charm) - better routing - made first real prototype board (self etching) - board works great with Zentris software
Parts:
- removed PAD1, PAD2: (no value), wirepad:2,54/1,0
- removed R2: ca 100k, rcl:R-EU_R0603
- added LSP1, LSP2: LSP11, solpad:LSP11
- added R1TRIM: 500K, rcl:R-TRIMM3374
- renumbered 13,3V-2GND to 3,3V-2GND
Connections:
- net N$7: now also LSP2.MP; no longer PAD2.P
- net N$8: now also R1TRIM.S; no longer R2.1
- net N$9: now also LSP1.MP, R1TRIM.A; no longer PAD1.P, R2.2
Other:
- moved on the sheet: 1RX-2TX, IC1E, IC1F, IC1P, PROG
Changed lines of the file:
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@@
 <?xml version="1.0" encoding="utf-8"?>
 <!DOCTYPE eagle SYSTEM "eagle.dtd">
-<eagle version="7.6.0">
+<eagle version="7.7.0">
 <drawing>
 <settings>
@@
 <parts>
 <part name="IC1" library="74xx-eu" deviceset="74*14" device="D" technology="HC"/>
-<part name="R2" library="rcl" deviceset="R-EU_" device="R0603" value="ca 100k"/>
 <part name="R3" library="rcl" deviceset="R-EU_" device="R0603" value="100"/>
 <part name="GND" library="pinhead" deviceset="PINHD-1X1" device=""/>
@@
 <part name="VIN" library="pinhead" deviceset="PINHD-1X1" device=""/>
 <part name="C4" library="capsmd" deviceset="C1206" device="" value="10µF"/>
-<part name="ESP" library="esp8266modules" deviceset="ESP12" device="" value=""/>
+<part name="ESP" library="esp8266modules" deviceset="ESP12" device="" value="ESP12"/>
 <part name="1RX-2TX" library="pinhead" deviceset="PINHD-1X2" device=""/>
 <part name="C1" library="cap-master" deviceset="CP-" device="SV-E/F" value="1000µF"/>
 <part name="PROG" library="switch-tact" deviceset="DTSM-6" device=""/>
 <part name="RESET" library="switch-tact" deviceset="DTSM-6" device=""/>
-<part name="PAD1" library="wirepad" deviceset="2,54/1,0" device=""/>
-<part name="PAD2" library="wirepad" deviceset="2,54/1,0" device=""/>
-<part name="13,3V-2GND" library="pinhead" deviceset="PINHD-1X2" device=""/>
+<part name="3,3V-2GND" library="pinhead" deviceset="PINHD-1X2" device=""/>
+<part name="LSP1" library="solpad" deviceset="LSP11" device=""/>
+<part name="LSP2" library="solpad" deviceset="LSP11" device=""/>
+<part name="R1TRIM" library="rcl" deviceset="R-TRIMM" device="3374" value="500K"/>
 </parts>
 <sheets>
@@
 <instance part="IC1" gate="C" x="111.76" y="116.84"/>
 <instance part="IC1" gate="D" x="55.88" y="167.64"/>
-<instance part="IC1" gate="E" x="76.2" y="167.64"/>
-<instance part="IC1" gate="F" x="96.52" y="167.64"/>
-<instance part="IC1" gate="P" x="177.8" y="106.68"/>
-<instance part="R2" gate="G$1" x="68.58" y="132.08" rot="R90"/>
+<instance part="IC1" gate="E" x="83.82" y="167.64"/>
+<instance part="IC1" gate="F" x="114.3" y="167.64"/>
+<instance part="IC1" gate="P" x="185.42" y="99.06" rot="R90"/>
 <instance part="R3" gate="G$1" x="132.08" y="116.84" rot="R180"/>
 <instance part="GND" gate="G$1" x="22.86" y="50.8" rot="R180"/>
@@
 <instance part="C4" gate="G$1" x="35.56" y="73.66"/>
 <instance part="ESP" gate="G$1" x="134.62" y="83.82"/>
-<instance part="1RX-2TX" gate="G$1" x="165.1" y="88.9"/>
+<instance part="1RX-2TX" gate="G$1" x="167.64" y="127"/>
 <instance part="C1" gate="G$1" x="111.76" y="68.58" rot="R90"/>
-<instance part="PROG" gate="G$1" x="177.8" y="78.74"/>
+<instance part="PROG" gate="G$1" x="185.42" y="78.74"/>
 <instance part="RESET" gate="G$1" x="101.6" y="88.9"/>
-<instance part="PAD1" gate="P" x="129.54" y="144.78" rot="R180"/>
-<instance part="PAD2" gate="P" x="129.54" y="134.62" rot="R180"/>
-<instance part="13,3V-2GND" gate="G$1" x="91.44" y="48.26" rot="R270"/>
+<instance part="3,3V-2GND" gate="G$1" x="91.44" y="48.26" rot="R270"/>
+<instance part="LSP1" gate="1" x="132.08" y="144.78" rot="R270"/>
+<instance part="LSP2" gate="1" x="132.08" y="134.62" rot="R270"/>
+<instance part="R1TRIM" gate="G$1" x="68.58" y="134.62" rot="R270"/>
 </instances>
 <busses>
@@
 <pinref part="IC1" gate="D" pin="O"/>
 <pinref part="IC1" gate="E" pin="I"/>
+<wire x1="73.66" y1="167.64" x2="66.04" y2="167.64" width="0.1524" layer="91"/>
 </segment>
 </net>
@@
 <pinref part="IC1" gate="E" pin="O"/>
 <pinref part="IC1" gate="F" pin="I"/>
+<wire x1="104.14" y1="167.64" x2="93.98" y2="167.64" width="0.1524" layer="91"/>
 </segment>
 </net>
@@
 <junction x="154.94" y="73.66"/>
 <pinref part="PROG" gate="G$1" pin="1"/>
-<wire x1="154.94" y1="73.66" x2="177.8" y2="73.66" width="0.1524" layer="91"/>
+<wire x1="154.94" y1="73.66" x2="185.42" y2="73.66" width="0.1524" layer="91"/>
 <pinref part="RESET" gate="G$1" pin="1"/>
 <wire x1="101.6" y1="83.82" x2="101.6" y2="60.96" width="0.1524" layer="91"/>
 <junction x="101.6" y="60.96"/>
 <pinref part="PROG" gate="G$1" pin="2"/>
-<wire x1="177.8" y1="73.66" x2="180.34" y2="73.66" width="0.1524" layer="91"/>
-<wire x1="154.94" y1="68.58" x2="187.96" y2="68.58" width="0.1524" layer="91"/>
+<wire x1="185.42" y1="73.66" x2="187.96" y2="73.66" width="0.1524" layer="91"/>
+<wire x1="154.94" y1="68.58" x2="200.66" y2="68.58" width="0.1524" layer="91"/>
 <junction x="154.94" y="68.58"/>
-<wire x1="187.96" y1="68.58" x2="187.96" y2="93.98" width="0.1524" layer="91"/>
-<wire x1="187.96" y1="93.98" x2="177.8" y2="93.98" width="0.1524" layer="91"/>
+<wire x1="200.66" y1="68.58" x2="200.66" y2="99.06" width="0.1524" layer="91"/>
 <pinref part="IC1" gate="P" pin="GND"/>
-<wire x1="177.8" y1="93.98" x2="177.8" y2="99.06" width="0.1524" layer="91"/>
-<pinref part="13,3V-2GND" gate="G$1" pin="2"/>
+<wire x1="200.66" y1="99.06" x2="193.04" y2="99.06" width="0.1524" layer="91"/>
+<pinref part="3,3V-2GND" gate="G$1" pin="2"/>
 <wire x1="91.44" y1="60.96" x2="91.44" y2="50.8" width="0.1524" layer="91"/>
 <junction x="91.44" y="60.96"/>
@@
 <net name="N$8" class="0">
 <segment>
-<wire x1="68.58" y1="127" x2="68.58" y2="116.84" width="0.1524" layer="91"/>
 <wire x1="68.58" y1="116.84" x2="66.04" y2="116.84" width="0.1524" layer="91"/>
 <wire x1="73.66" y1="116.84" x2="68.58" y2="116.84" width="0.1524" layer="91"/>
 <junction x="68.58" y="116.84"/>
-<pinref part="R2" gate="G$1" pin="1"/>
 <pinref part="IC1" gate="A" pin="O"/>
 <pinref part="IC1" gate="B" pin="I"/>
+<pinref part="R1TRIM" gate="G$1" pin="S"/>
+<wire x1="68.58" y1="129.54" x2="68.58" y2="116.84" width="0.1524" layer="91"/>
 </segment>
 </net>
@@
 <wire x1="116.84" y1="86.36" x2="111.76" y2="86.36" width="0.1524" layer="91"/>
 <junction x="111.76" y="86.36"/>
-<pinref part="13,3V-2GND" gate="G$1" pin="1"/>
+<pinref part="3,3V-2GND" gate="G$1" pin="1"/>
 <wire x1="93.98" y1="73.66" x2="93.98" y2="50.8" width="0.1524" layer="91"/>
 <junction x="93.98" y="73.66"/>
@@
 <pinref part="ESP" gate="G$1" pin="TX"/>
 <pinref part="1RX-2TX" gate="G$1" pin="1"/>
-<wire x1="149.86" y1="91.44" x2="162.56" y2="91.44" width="0.1524" layer="91"/>
+<wire x1="149.86" y1="91.44" x2="160.02" y2="91.44" width="0.1524" layer="91"/>
+<wire x1="160.02" y1="91.44" x2="160.02" y2="129.54" width="0.1524" layer="91"/>
+<wire x1="160.02" y1="129.54" x2="165.1" y2="129.54" width="0.1524" layer="91"/>
 </segment>
 </net>
@@
 <pinref part="1RX-2TX" gate="G$1" pin="2"/>
 <wire x1="149.86" y1="88.9" x2="162.56" y2="88.9" width="0.1524" layer="91"/>
+<wire x1="162.56" y1="88.9" x2="162.56" y2="127" width="0.1524" layer="91"/>
+<wire x1="162.56" y1="127" x2="165.1" y2="127" width="0.1524" layer="91"/>
 </segment>
 </net>
@@
 <segment>
 <pinref part="ESP" gate="G$1" pin="GPIO0"/>
-<wire x1="149.86" y1="81.28" x2="177.8" y2="83.82" width="0.1524" layer="91"/>
+<wire x1="149.86" y1="81.28" x2="182.88" y2="81.28" width="0.1524" layer="91"/>
+<wire x1="182.88" y1="81.28" x2="185.42" y2="83.82" width="0.1524" layer="91"/>
 <pinref part="PROG" gate="G$1" pin="3"/>
 <pinref part="PROG" gate="G$1" pin="4"/>
-<wire x1="177.8" y1="83.82" x2="180.34" y2="83.82" width="0.1524" layer="91"/>
-<junction x="177.8" y="83.82"/>
-</segment>
-<segment>
-<wire x1="40.64" y1="144.78" x2="40.64" y2="116.84" width="0.1524" layer="91"/>
+<wire x1="185.42" y1="83.82" x2="187.96" y2="83.82" width="0.1524" layer="91"/>
+<junction x="185.42" y="83.82"/>
+</segment>
+<segment>
+<wire x1="40.64" y1="144.78" x2="40.64" y2="134.62" width="0.1524" layer="91"/>
+<wire x1="40.64" y1="134.62" x2="40.64" y2="116.84" width="0.1524" layer="91"/>
 <wire x1="40.64" y1="116.84" x2="45.72" y2="116.84" width="0.1524" layer="91"/>
-<wire x1="127" y1="144.78" x2="68.58" y2="144.78" width="0.1524" layer="91"/>
+<wire x1="129.54" y1="144.78" x2="40.64" y2="144.78" width="0.1524" layer="91"/>
 <pinref part="IC1" gate="A" pin="I"/>
-<pinref part="R2" gate="G$1" pin="2"/>
-<wire x1="68.58" y1="144.78" x2="40.64" y2="144.78" width="0.1524" layer="91"/>
-<wire x1="68.58" y1="137.16" x2="68.58" y2="144.78" width="0.1524" layer="91"/>
-<junction x="68.58" y="144.78"/>
-<pinref part="PAD1" gate="P" pin="P"/>
+<pinref part="LSP1" gate="1" pin="MP"/>
+<pinref part="R1TRIM" gate="G$1" pin="A"/>
+<wire x1="63.5" y1="134.62" x2="40.64" y2="134.62" width="0.1524" layer="91"/>
+<junction x="40.64" y="134.62"/>
 </segment>
 </net>
@@
 <pinref part="IC1" gate="B" pin="O"/>
 <pinref part="IC1" gate="C" pin="I"/>
-<pinref part="PAD2" gate="P" pin="P"/>
-<wire x1="127" y1="134.62" x2="99.06" y2="134.62" width="0.1524" layer="91"/>
+<wire x1="129.54" y1="134.62" x2="99.06" y2="134.62" width="0.1524" layer="91"/>
+<pinref part="LSP2" gate="1" pin="MP"/>
 </segment>
 </net>
@@
 <pinref part="ESP" gate="G$1" pin="GPIO4"/>
 <wire x1="149.86" y1="86.36" x2="170.18" y2="86.36" width="0.1524" layer="91"/>
-<wire x1="170.18" y1="86.36" x2="170.18" y2="119.38" width="0.1524" layer="91"/>
-<wire x1="170.18" y1="119.38" x2="177.8" y2="119.38" width="0.1524" layer="91"/>
+<wire x1="170.18" y1="86.36" x2="170.18" y2="99.06" width="0.1524" layer="91"/>
+<wire x1="170.18" y1="99.06" x2="177.8" y2="99.06" width="0.1524" layer="91"/>
 <pinref part="IC1" gate="P" pin="VCC"/>
-<wire x1="177.8" y1="119.38" x2="177.8" y2="114.3" width="0.1524" layer="91"/>
-</segment>
-</net>
+</segment>
+</net>

Commit message: updated readme
Parts:
- renumbered 3,3V-2GND to GND-3.3V
Changed lines of the file:
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@@
 <part name="PROG" library="switch-tact" deviceset="DTSM-6" device=""/>
 <part name="RESET" library="switch-tact" deviceset="DTSM-6" device=""/>
-<part name="3,3V-2GND" library="pinhead" deviceset="PINHD-1X2" device=""/>
+<part name="GND-3.3V" library="pinhead" deviceset="PINHD-1X2" device=""/>
 <part name="LSP1" library="solpad" deviceset="LSP11" device=""/>
 <part name="LSP2" library="solpad" deviceset="LSP11" device=""/>
@@
 <instance part="PROG" gate="G$1" x="185.42" y="78.74"/>
 <instance part="RESET" gate="G$1" x="101.6" y="88.9"/>
-<instance part="3,3V-2GND" gate="G$1" x="91.44" y="48.26" rot="R270"/>
+<instance part="GND-3.3V" gate="G$1" x="91.44" y="48.26" rot="R270"/>
 <instance part="LSP1" gate="1" x="132.08" y="144.78" rot="R270"/>
 <instance part="LSP2" gate="1" x="132.08" y="134.62" rot="R270"/>
@@
 <pinref part="IC1" gate="P" pin="GND"/>
 <wire x1="200.66" y1="99.06" x2="193.04" y2="99.06" width="0.1524" layer="91"/>
-<pinref part="3,3V-2GND" gate="G$1" pin="2"/>
+<pinref part="GND-3.3V" gate="G$1" pin="2"/>
 <wire x1="91.44" y1="60.96" x2="91.44" y2="50.8" width="0.1524" layer="91"/>
 <junction x="91.44" y="60.96"/>
@@
 <wire x1="116.84" y1="86.36" x2="111.76" y2="86.36" width="0.1524" layer="91"/>
 <junction x="111.76" y="86.36"/>
-<pinref part="3,3V-2GND" gate="G$1" pin="1"/>
+<pinref part="GND-3.3V" gate="G$1" pin="1"/>
 <wire x1="93.98" y1="73.66" x2="93.98" y2="50.8" width="0.1524" layer="91"/>
 <junction x="93.98" y="73.66"/>
