File: sensor_v1.brd (EAGLE design)
At the start: 196.5 x 34.3 mm, 16 parts, among them IC1 74HC14D, IC2 HT7333

Commit message: reorder structure for more versions
Connections:
- net N$4: now also ESP.GPIO16
Routing:
- net N$4: track 35.1 -> 40.5 mm
Changed lines of the file:
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@@
 <wire x1="23.01385" y1="15.8496" x2="22.014484375" y2="15.7496" width="0.508" layer="1"/>
 <wire x1="22.014484375" y1="15.7496" x2="20.7264" y2="16.637684375" width="0.508" layer="1" curve="-90"/>
-<wire x1="28.448" y1="20.32" x2="24.659075" y2="16.531075" width="0.508" layer="1"/>
+<wire x1="28.448" y1="20.32" x2="25.5015" y2="17.3735" width="0.508" layer="1"/>
+<wire x1="25.5015" y1="17.3735" x2="24.659075" y2="16.531075" width="0.508" layer="1"/>
 <wire x1="24.659075" y1="16.531075" x2="23.01385" y2="15.8496" width="0.508" layer="1" curve="-45.000077"/>
 <wire x1="29.2608" y1="20.32" x2="28.448" y2="20.32" width="0.508" layer="1"/>
 <wire x1="11.7856" y1="30.48" x2="11.52" y2="30.245" width="0.508" layer="1"/>
 <wire x1="29.2608" y1="20.32" x2="29.47" y2="20.47" width="0.508" layer="1"/>
+<contactref element="ESP" pad="GPIO16"/>
+<wire x1="27.625" y1="14.55" x2="29.375" y2="14.5" width="0.508" layer="1"/>
+<wire x1="27.125" y1="15.25" x2="27.625" y2="14.55" width="0.508" layer="1"/>
+<wire x1="25.5015" y1="17.3735" x2="27.125" y2="15.25" width="0.508" layer="1"/>
+<wire x1="29.375" y1="14.5" x2="29.47" y2="14.47" width="0.508" layer="1"/>
 </signal>
 <signal name="N$7">
