File: sensor_v1.sch (EAGLE design)
At the start: 16 parts, among them IC1 74HC14D, IC2 HT7333

Commit message: reorder structure for more versions
Connections:
- net N$4: now also ESP.GPIO16
Changed lines of the file:
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@@
 <wire x1="104.14" y1="93.98" x2="116.84" y2="93.98" width="0.1524" layer="91"/>
 <wire x1="116.84" y1="93.98" x2="116.84" y2="91.44" width="0.1524" layer="91"/>
+<pinref part="ESP" gate="G$1" pin="GPIO16"/>
+<wire x1="116.84" y1="83.82" x2="116.84" y2="91.44" width="0.1524" layer="91"/>
+<junction x="116.84" y="91.44"/>
 </segment>
 </net>
